File: hardware/esp-usb/esp-usb.kicad_pcb (KiCad board)
At the start: 2 copper layers, 22 x 14.1 mm, 5 parts, among them J1 USB_A, U1 ESP32-C3, U7 TPD2EUSB30A

Commit message: beta version!
Parts:
- added AE1: Antenna, RF_Antenna:Johanson_2450AT18x100, F.Cu at (114.4, 90.3)
- added C10: 10pF, Capacitor_SMD:C_0402_1005Metric, F.Cu at (110.7, 93.7)
- added C12: 1uF, Capacitor_SMD:C_0402_1005Metric, F.Cu at (102.6, 95.3)
- added C3: 1pF, Capacitor_SMD:C_0402_1005Metric, F.Cu at (108.0, 86.7)
- added C4: 1pF, Capacitor_SMD:C_0402_1005Metric, F.Cu at (110.8, 85.8)
- added C5: 10nF, Capacitor_SMD:C_0402_1005Metric, F.Cu at (105.4, 86.2)
- added C6: 10nF, Capacitor_SMD:C_0402_1005Metric, F.Cu at (103.6, 86.2)
- added C7: 1uF, Capacitor_SMD:C_0402_1005Metric, F.Cu at (104.8, 94.5)
- added C8: 10nF, Capacitor_SMD:C_0402_1005Metric, F.Cu at (103.9, 94.5)
- added C9: 10pF, Capacitor_SMD:C_0402_1005Metric, F.Cu at (111.8, 88.8)
- added D1: LED, LED_SMD:LED_0603_1608Metric, F.Cu at (107.3, 94.6)
- added D2: LED, LED_SMD:LED_0603_1608Metric, F.Cu at (99.6, 87.2)
- added J2: Conn_01x05, Connector_PinHeader_2.54mm:PinHeader_1x05_P2.54mm_Vertical, F.Cu at (100.5, 98.0)
- added J3: Conn_01x05, Connector_PinHeader_2.54mm:PinHeader_1x05_P2.54mm_Vertical, F.Cu at (100.5, 82.8)
- added L1: 2.4nH, Inductor_SMD:L_0402_1005Metric, F.Cu at (109.4, 86.3)
- added R1: 0, Resistor_SMD:R_0402_1005Metric, F.Cu at (110.3, 89.2)
- added R2: 4.7k, Resistor_SMD:R_0402_1005Metric, F.Cu at (102.0, 86.2)
- added R3: 4.7k, Resistor_SMD:R_0402_1005Metric, F.Cu at (108.5, 94.7)
- added SW1: SW_Push, Button_Switch_SMD:SW_SPST_B3U-1000P, F.Cu at (99.7, 90.3)
- added U2: SPX3819M5-L-3-3, Package_TO_SOT_SMD:SOT-23-5, F.Cu at (100.1, 94.5)
- added Y1: Crystal_GND23, Crystal:Crystal_SMD_2520-4Pin_2.5x2.0mm, F.Cu at (111.0, 91.5)
- moved C2 10.7 mm to (108.9, 88.5), turned to 90 degrees
- moved C1 10.2 mm to (108.0, 88.5), turned to 90 degrees
- moved U7 4.90 mm to (100.0, 85.7)
- moved U1 1.62 mm to (104.4, 90.3), turned to -90 degrees
Connections:
- U1 pad 1: unconnected-(U1-LNA_IN-Pad1) -> /LNA_IN
- U1 pad 10: unconnected-(U1-MTDI-Pad10) -> /GPIO5
- U1 pad 12: unconnected-(U1-MTCK-Pad12) -> /GPIO6
- U1 pad 13: unconnected-(U1-MTDO-Pad13) -> /GPIO7
- U1 pad 16: unconnected-(U1-GPIO10-Pad16) -> /GPIO10
- U1 pad 27: unconnected-(U1-U0RXD-Pad27) -> /GPIO20
- U1 pad 28: unconnected-(U1-U0TXD-Pad28) -> /GPIO21
- U1 pad 29: unconnected-(U1-XTAL_N-Pad29) -> /XA
- U1 pad 30: unconnected-(U1-XTAL_P-Pad30) -> Net-(U1-XTAL_P)
- U1 pad 4: unconnected-(U1-XTAL_32K_P-Pad4) -> /GPIO0
- U1 pad 5: unconnected-(U1-XTAL_32K_N-Pad5) -> /GPIO1
- U1 pad 7: unconnected-(U1-CHIP_EN-Pad7) -> +3V3
- U1 pad 8: unconnected-(U1-GPIO3-Pad8) -> /GPIO3
- U1 pad 9: unconnected-(U1-MTMS-Pad9) -> /GPIO4
Routing:
- net /D+: track 7.61 -> 27.9 mm, vias 0 -> 2
- net /D-: track 7.61 -> 27.8 mm, vias 0 -> 2
- net +5V: track 0.00 -> 16.8 mm
- net /GPIO5: track 0.00 -> 13.6 mm, vias 0 -> 2
- net /GPIO7: track 0.00 -> 11.3 mm, vias 0 -> 2
- net /GPIO21: track 0.00 -> 10.1 mm
- net /GPIO0: track 0.00 -> 9.94 mm
- net /GPIO20: track 0.00 -> 9.39 mm
- net /GPIO1: track 0.00 -> 7.94 mm
- net /XA: track 0.00 -> 7.68 mm
- net /GPIO3: track 0.00 -> 6.66 mm
- net /GPIO10: track 0.00 -> 6.52 mm
- net /GPIO6: track 0.00 -> 6.32 mm
- net /GPIO4: track 0.00 -> 6.31 mm
- net +3V3: track 0.00 -> 5.18 mm, vias 0 -> 14
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- added copper zone on In2.Cu, net +3V3
- added copper zone on In1.Cu, net GND
- removed copper zone on F.Cu, net +5V
Other:
- board size 22 x 14.1 mm -> 30 x 18 mm
- copper layers 2 -> 4

Commit message: Rev 3 ig
Parts:
- removed C1: 1uF, Capacitor_SMD:C_0402_1005Metric
- added C11: 1uF, Capacitor_SMD:C_0402_1005Metric, F.Cu at (100.2, 90.3)
- added C13: 100nF, Capacitor_SMD:C_0402_1005Metric, F.Cu at (99.2, 95.8)
- added F1: 5+V, Fuse:Fuse_0603_1608Metric, F.Cu at (97.8, 92.9)
- added J4: USB_A, esp-usb-lib:USBPCB, B.Cu at (95.0, 90.4)
- C2, C5, C6: value 10nF -> 100nF
- C8: value 10nF -> 1uF
- R1: value 0 -> 10k
- R2, R3: value 4.7k -> 1k
- Y1: footprint Crystal:Crystal_SMD_2520-4Pin_2.5x2.0mm -> Crystal:Crystal_SMD_2016-4Pin_2.0x1.6mm
- moved D2 10.1 mm to (109.6, 85.4)
- moved R3 8.88 mm to (107.1, 85.9), turned to 180 degrees
- moved C6 8.09 mm to (110.0, 91.2), turned to 0 degrees
- moved D1 8.07 mm to (109.6, 86.9), turned to 0 degrees
- moved C8 7.85 mm to (110.0, 89.5), turned to 0 degrees
- moved C7 6.80 mm to (101.9, 88.3), turned to 180 degrees
- moved C9 6.29 mm to (110.1, 94.8), turned to 0 degrees
- moved L1 6.04 mm to (110.9, 92.1)
- moved C3 6.03 mm to (109.5, 92.5)
- moved C4 6.00 mm to (112.3, 91.6)
- moved C2 5.51 mm to (110.1, 93.9), turned to 0 degrees
- moved R2 5.35 mm to (107.2, 85.0), turned to 180 degrees
- moved U7 5.24 mm to (97.8, 90.4)
- moved SW1 4.89 mm to (102.2, 86.2), turned to 180 degrees
- moved Y1 4.74 mm to (107.7, 94.8), turned to 0 degrees
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Connections:
- C8 pad 1: +3V3 -> Net-(U1-CHIP_EN)
- D1 pad 1: /GPIO7 -> /GPIO3
- D2 pad 1: /GPIO6 -> /GPIO4
- J1 pad 1: +5V -> Net-(J1-VBUS)
- J2 pad 2: /GPIO10 -> /GPIO7
- J2 pad 3: /GPIO5 -> /GPIO10
- J3 pad 2: /GPIO4 -> /GPIO6
- J3 pad 3: /GPIO3 -> /GPIO5
- R1 pad 1: Net-(U1-XTAL_P) -> +3V3
- R1 pad 2: /XB -> Net-(U1-CHIP_EN)
- R2 pad 2: +3V3 -> GND
- R3 pad 2: +3V3 -> GND
- U1 pad 30: Net-(U1-XTAL_P) -> /XB
- U1 pad 7: +3V3 -> Net-(U1-CHIP_EN)
- U2 pad 4: unconnected-(U2-BP-Pad4) -> Net-(U2-BP)
Routing:
- net +3V3: track 5.18 -> 32.6 mm, vias 14 -> 8
- net Net-(J1-VBUS): track 0.00 -> 21.4 mm, vias 0 -> 2
- net +5V: track 16.8 -> 4.94 mm
- net /GPIO5: track 13.6 -> 6.09 mm
- net /GPIO10: track 6.52 -> 13.1 mm, vias 0 -> 2
- net /GPIO7: track 11.3 -> 16.6 mm
- net /GPIO3: track 6.66 -> 1.90 mm
- net /GPIO1: track 7.94 -> 11.6 mm
- net /D-: track 27.8 -> 24.3 mm, vias 2 -> 3
- net /GPIO4: track 6.31 -> 2.97 mm
- net Net-(U1-XTAL_P): track 3.12 -> 0.00 mm
- net Net-(AE1-A): track 4.75 -> 1.67 mm
- net /GPIO20: track 9.39 -> 6.97 mm
- net Net-(D1-A): track 1.28 -> 3.33 mm, vias 0 -> 2
- net /D+: track 27.9 -> 26.1 mm, vias 2 -> 3
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- removed copper zone on In2.Cu, net +3V3
- removed copper zone on In1.Cu, net GND
Other:
- copper layers 4 -> 2
