File: hardware/esp-usb/esp-usb.kicad_sch (KiCad schematic)
At the start: 10 parts, among them J1 USB_A, SW1 SW_Push, U1 ESP32-C3, U7 TPD2EUSB30A

Commit message: beta version!
Parts:
- added C10, C9: 10pF, Capacitor_SMD:C_0402_1005Metric, symbol Device:C_Small
- added C12, C7: 1uF, Capacitor_SMD:C_0402_1005Metric, symbol Device:C_Small
- added C5, C6, C8: 10nF, Capacitor_SMD:C_0402_1005Metric, symbol Device:C_Small
- added D1, D2: LED, LED_SMD:LED_0603_1608Metric, symbol Device:LED
- added J2, J3: Conn_01x05, Connector_PinHeader_2.54mm:PinHeader_1x05_P2.54mm_Vertical, symbol Connector_Generic:Conn_01x05
- added R1: 0, Resistor_SMD:R_0402_1005Metric, symbol Device:R_Small
- added R2, R3: 4.7k, Resistor_SMD:R_0402_1005Metric, symbol Device:R_Small
- added U2: SPX3819M5-L-3-3, Package_TO_SOT_SMD:SOT-23-5, symbol Regulator_Linear:SPX3819M5-L-3-3
- added Y1: Crystal_GND23, Crystal:Crystal_SMD_2520-4Pin_2.5x2.0mm, symbol Device:Crystal_GND24
- AE1: footprint (none) -> RF_Antenna:Johanson_2450AT18x100; LCSC Part # (none) -> C89334
- L1: value L -> 2.4nH; footprint (none) -> Inductor_SMD:L_0402_1005Metric; LCSC Part # (none) -> C142237
- SW1: footprint (none) -> Button_Switch_SMD:SW_SPST_B3U-1000P; LCSC Part # (none) -> C2689695
Connections:
- net +3V3: now also C12.1, C5.1, C6.1, C7.1, C8.1, J2.1 (Pin_1), R2.2, R3.2, U2.5 (OUT)
- net +5V: now also U2.1 (IN), U2.3 (EN)
- net GND: now also C10.2, C12.2, C5.2, C6.2, C7.2, C8.2, C9.2, J3.1 (Pin_1), U2.2 (GND), Y1.2, Y1.4
- net GPIO3: now also J3.3 (Pin_3)
- net GPIO4: now also J3.2 (Pin_2)
- net GPIO5: now also J2.3 (Pin_3)
- net GPIO6: now also D2.1 (K)
- net GPIO7: now also D1.1 (K)
- net GPIO10: now reaches U1.16 (GPIO10)
- net GPIO10: now also J2.2 (Pin_2)
- net GPIO20: now reaches U1.27 (U0RXD)
- net GPIO20: now also J2.4 (Pin_4)
- net GPIO21: now reaches U1.28 (U0TXD)
- net GPIO21: now also J2.5 (Pin_5)
- net XA: now reaches U1.29 (XTAL_N)
- net XA: now also C10.1, Y1.1
- net at U1.30 (XTAL_P): now also R1.1
- net GPIO0: now reaches U1.4 (XTAL_32K_P)
- net GPIO0: now also J3.5 (Pin_5)
- net GPIO1: now reaches U1.5 (XTAL_32K_N)
- net GPIO1: now also J3.4 (Pin_4)
- new net: D1.2 (A), R3.1
- new net: D2.2 (A), R2.1
- new net XB: C9.1, R1.2, Y1.3
- no-connect marks 6 -> 7
Other:
- note added: "2.4GHz Antenna"
- note added: "Core"
- note added: "Crystal"
- note added: "GPIO"
- note added: "LDO"
- note added: "User LEDs"
- company: (none) -> Chengyin Yao
- title: (none) -> ECP USB
- moved on the sheet: AE1, C1, C2, C3, C4, J1, L1, SW1, U1, U7

Commit message: Rev 3 ig
Parts:
- removed C1: 1uF, Capacitor_SMD:C_0402_1005Metric, symbol Device:C_Small
- added C11: 1uF, Capacitor_SMD:C_0402_1005Metric, symbol Device:C_Small
- added C13: 100nF, Capacitor_SMD:C_0402_1005Metric, symbol Device:C_Small
- added F1: 5+V, Fuse:Fuse_0603_1608Metric, symbol Device:Polyfuse_Small
- added J4: USB_A, esp-usb-lib:USBPCB, symbol Connector:USB_A
- AE1: LCSC Part # C89334 -> C127629
- C10, C9: LCSC Part # (none) -> C32949
- C2, C5, C6: value 10nF -> 100nF; LCSC Part # C15195 -> (none)
- C8: value 10nF -> 1uF; LCSC Part # C15195 -> C52923
- R1: value 0 -> 10k
- R2, R3: value 4.7k -> 1k; LCSC Part # (none) -> C11702
- Y1: footprint Crystal:Crystal_SMD_2520-4Pin_2.5x2.0mm -> Crystal:Crystal_SMD_2016-4Pin_2.0x1.6mm; LCSC Part # C2885592 -> C424432
Connections:
- net +3V3: now also R1.1; no longer C8.1, R2.2, R3.2, U1.7 (CHIP_EN)
- net +5V: now also C11.1, F1.2; no longer J1.1 (VBUS)
- net D+: now also J4.3 (D+)
- net D-: now also J4.2 (D-)
- net GND: now also R2.2, R3.2, C11.2, C13.2, J4.4 (GND)
- net GPIO10: now also J2.3 (Pin_3); no longer J2.2 (Pin_2)
- net GPIO3: now also D1.1 (K); no longer J3.3 (Pin_3)
- net GPIO4: now also D2.1 (K); no longer J3.2 (Pin_2)
- net GPIO5: now also J3.3 (Pin_3); no longer J2.3 (Pin_3)
- net GPIO6: now also J3.2 (Pin_2); no longer D2.1 (K)
- net GPIO7: now also J2.2 (Pin_2); no longer D1.1 (K)
- net XB: now also U1.30 (XTAL_P); no longer R1.2
- net at U2.4 (BP): now also C13.1
- new net: F1.1, J1.1 (VBUS), J4.1 (VBUS)
- new net: C8.1, R1.2, U1.7 (CHIP_EN)
- no-connect marks 7 -> 6
Other:
- note removed: "Boot Select"
- moved on the sheet: AE1, C12, C2, C3, C4, C5, C6, C7, C8, J1, L1, SW1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
