File: hardware/esp-usb.kicad_pcb (KiCad board)
At the start: 2 copper layers, 30 x 18 mm, 29 parts, among them J1 USB_A, J2 Conn_01x05, J3 Conn_01x05, J4 USB_A, SW1 SW_Push, U1 ESP32-C3, U2 SPX3819M5-L-3-3, U7 TPD2EUSB30A, Y1 Crystal_GND23

Commit message: Final rev!
Parts:
- moved C8 1.18 mm to (110.0, 88.3)
- moved R1 0.97 mm to (110.0, 89.5)
- moved R2 0.10 mm to (107.1, 85.0)
- moved F1 0.06 mm to (97.7, 92.9)
Routing:
- net Net-(U1-CHIP_EN): track 0.00 -> 3.23 mm
- net Net-(J1-VBUS): track 21.4 -> 20.2 mm
- net /D+: track 26.1 -> 25.6 mm
- net GND: vias 54 -> 57
